Commit message: Update megarover_description for gazebo and ROS2

File: urdf/f120a.xacro (robot description, xacro)
@@ -1,6 +1,7 @@
 <?xml version="1.0"?>
 <robot name="f120a" xmlns:xacro="http://www.ros.org/wiki/xacro">
-  <xacro:include filename="$(find megarover_description)/urdf/f120a_base_model.xacro" />
+  <xacro:include filename="$(find megarover_description)/urdf/materials.xacro" />
   <xacro:include filename="$(find megarover_description)/urdf/f120a.gazebo" />
+  <xacro:include filename="$(find megarover_description)/urdf/f120a_ros2_control.xacro" />
   <!-- OPTION  LRF TG30 -->
   <!-- <xacro:include filename="$(find vs_rover_options_description)/urdf/lrf/tg30_f120a.xacro" /> -->
@@ -23,3 +24,87 @@
     <child link="link0_1" />
   </joint> -->
+  <link name="base_footprint" />
+  <joint name="base_joint" type="fixed">
+    <parent link="base_footprint" />
+    <child link="base_link" />
+    <origin xyz="-0.108 0 0" rpy="0 0 -1.5708" />
+  </joint>
+  <link name="base_link">
+    <inertial>
+      <origin xyz="-0.000002 -0.012552 0.124849" rpy="0 0 0" />
+      <mass value="26.5" />
+      <inertia ixx="3.703059e-01" iyy="2.862913e-01" izz="5.773479e-01"
+        ixy="1.109256e-05" iyz="4.327049e-03"
+        ixz="-8.886529e-07" />
+    </inertial>
+    <visual>
+      <origin xyz="0 0 0" rpy="0 0 0" />
+      <geometry>
+        <mesh filename="package://megarover_description/meshes/f120a/base_link.stl" scale="0.001 0.001 0.001" />
+      </geometry>
+      <material name="silver" />
+    </visual>
+    <collision>
+      <origin xyz="0 0 0" rpy="0 0 0" />
+      <geometry>
+        <mesh filename="package://megarover_description/meshes/f120a/base_link.stl" scale="0.001 0.001 0.001" />
+      </geometry>
+    </collision>
+  </link>
+  <joint name="right_wheel_joint" type="continuous">
+    <origin xyz="0.202 0.108 0.085" rpy="0 -1.5708 0" />
+    <parent link="base_link" />
+    <child link="right_wheel_1" />
+    <axis xyz="0.0 0.0 1.0" />
+  </joint>
+  <link name="right_wheel_1">
+    <inertial>
+      <origin xyz="0.204466 0.108001 0.085004" rpy="0 0 0" />
+      <mass value="3.3" />
+      <inertia ixx="1.037325e-02" iyy="6.022157e-03" izz="6.021823e-03"
+        ixy="3.443741e-09" iyz="-1.410248e-07"
+        ixz="3.078066e-08" />
+    </inertial>
+    <visual>
+      <origin xyz="-0.085 -0.108 0.202" rpy="0 1.5708 0" />
+      <geometry>
+        <mesh filename="package://megarover_description/meshes/f120a/right_wheel_1.stl" scale="0.001 0.001 0.001" />
+      </geometry>
+      <material name="dark_grey" />
+    </visual>
+    <collision>
+      <origin xyz="-0.085 -0.108 0.202" rpy="0 1.5708 0" />
+      <geometry>
+        <mesh filename="package://megarover_description/meshes/f120a/right_wheel_1.stl" scale="0.001 0.001 0.001" />
+      </geometry>
+    </collision>
+  </link>
+  <joint name="left_wheel_joint" type="continuous">
+    <origin xyz="-0.202 0.108 0.085" rpy="0 -1.5708 0" />
+    <parent link="base_link" />
+    <child link="left_wheel_1" />
+    <axis xyz="0.0 0.0 1.0" />
+  </joint>
+  <link name="left_wheel_1">
+    <inertial>
+      <origin xyz="-0.204466 0.108004 0.085001" rpy="0 0 0" />
+      <mass value="3.3" />
+      <inertia ixx="1.037325e-02" iyy="6.021823e-03" izz="6.022157e-03"
+        ixy="-3.081416e-08" iyz="-1.410216e-07"
+        ixz="-3.441302e-09" />
+    </inertial>
+    <visual>
+      <origin xyz="-0.085 -0.108 -0.202" rpy="0 1.5708 0" />
+      <geometry>
+        <mesh filename="package://megarover_description/meshes/f120a/left_wheel_1.stl" scale="0.001 0.001 0.001" />
+      </geometry>
+      <material name="dark_grey" />
+    </visual>
+    <collision>
+      <origin xyz="-0.085 -0.108 -0.202" rpy="0 1.5708 0" />
+      <geometry>
+        <mesh filename="package://megarover_description/meshes/f120a/left_wheel_1.stl" scale="0.001 0.001 0.001" />
+      </geometry>
+    </collision>
+  </link>
 </robot>

File: urdf/mega3.xacro (robot description, xacro)
@@ -2,18 +2,20 @@
 <robot name="mega3" xmlns:xacro="http://www.ros.org/wiki/xacro">
   <xacro:include filename="$(find megarover_description)/urdf/materials.xacro" />
-  <xacro:include filename="$(find megarover_description)/urdf/mega3_base_model.xacro" />
   <xacro:include filename="$(find megarover_description)/urdf/mega3.gazebo" />
   <xacro:include filename="$(find megarover_description)/urdf/mega3_ros2_control.xacro" />
   <!-- OPTION LRF TG30 -->
-  <xacro:include filename="$(find vs_rover_options_description)/urdf/lrf/tg30_mega3.xacro" />
-  <!-- <xacro include filename="$(find vs_rover_options_description)/urdf/bumper/bumper_mega3.xacro" />
+  <!-- <xacro:include filename="$(find vs_rover_options_description)/urdf/lrf/tg30_mega3.xacro" /> -->
+  <!-- OPTION  bumper sensor -->
+  <!-- <xacro:include filename="$(find vs_rover_options_description)/urdf/bumper/bumper_mega3.xacro" />
   <xacro:bumperbaseboard prefix="front" parent="base_link" xyz="0 0.19 0.02" z_dir="180" />
   <xacro:bumperbaseboard prefix="back" parent="base_link" xyz="0 -0.19 0.02" z_dir="0" /> -->
-  <!-- <xacro include filename="$(find vs_rover_options_description)/urdf/cam_stay/cam_stay_mega3.xacro" />
+  <!-- OPTION  camera stay -->
+  <!-- <xacro:include filename="$(find vs_rover_options_description)/urdf/cam_stay/cam_stay_mega3.xacro" />
   <xacro:include filename="$(find vs_rover_options_description)/urdf/depth_cam/_d435i.urdf.xacro" />
   <xacro:sensor_d435i parent="cam_mount_link" use_nominal_extrinsics="true">
     <origin xyz="0.0295 0 0.0095" rpy="0 0 0" />
   </xacro:sensor_d435i> -->
-  <!-- <xacro include filename="$(find amir_description)/urdf/amir_for_rover.xacro" />
+  <!-- OPTION  AMIR 740 (disabled by default because of interference with camera stay)-->
+  <!-- <xacro:include filename="$(find amir_description)/urdf/amir_for_rover.xacro" />
   <joint name="base_fixed" type="fixed">
     <origin xyz="0.0 0.03 0.398" rpy="0 0 0" />
@@ -21,3 +23,87 @@
     <child link="link0_1" />
   </joint> -->
+  <link name="base_footprint" />
+  <joint name="base_joint" type="fixed">
+    <parent link="base_footprint" />
+    <child link="base_link" />
+    <origin xyz="-0.1 0 0" rpy="0 0 -1.5708" />
+  </joint>
+  <link name="base_link">
+    <inertial>
+      <origin xyz="0.000146 -0.000007 0.095171" rpy="0 0 0" />
+      <mass value="12" />
+      <inertia ixx="9.308603e-02" iyy="5.644759e-02" izz="1.250700e-01"
+        ixy="3.125032e-04" iyz="-2.464583e-03"
+        ixz="2.117978e-05" />
+    </inertial>
+    <visual>
+      <origin xyz="0 0 0" rpy="0 0 0" />
+      <geometry>
+        <mesh filename="package://megarover_description/meshes/mega3/base_link.stl" scale="0.001 0.001 0.001" />
+      </geometry>
+      <material name="silver" />
+    </visual>
+    <collision>
+      <origin xyz="0 0 0" rpy="0 0 0" />
+      <geometry>
+        <mesh filename="package://megarover_description/meshes/mega3/base_link.stl" scale="0.001 0.001 0.001" />
+      </geometry>
+    </collision>
+  </link>
+  <joint name="left_wheel_joint" type="continuous">
+    <origin xyz="-0.136 0.1 0.07" rpy="0 -1.5708 0" />
+    <parent link="base_link" />
+    <child link="left_wheel_1" />
+    <axis xyz="0.0 0.0 1.0" />
+  </joint>
+  <link name="left_wheel_1">
+    <inertial>
+      <origin xyz="-0.138454 0.100000 0.070000" rpy="0 0 0" />
+      <mass value="1.24" />
+      <inertia ixx="2.678186e-03" iyy="1.655435e-03" izz="1.655435e-03"
+        ixy="2.305704e-12" iyz="-5.140092e-11"
+        ixz="5.431314e-14" />
+    </inertial>
+    <visual>
+      <origin xyz="-0.07 -0.1 -0.136" rpy="0 1.5708 0" />
+      <geometry>
+        <mesh filename="package://megarover_description/meshes/mega3/left_wheel_1.stl" scale="0.001 0.001 0.001" />
+      </geometry>
+      <material name="dark_grey" />
+    </visual>
+    <collision>
+      <origin xyz="-0.07 -0.1 -0.136" rpy="0 1.5708 0" />
+      <geometry>
+        <mesh filename="package://megarover_description/meshes/mega3/left_wheel_1.stl" scale="0.001 0.001 0.001" />
+      </geometry>
+    </collision>
+  </link>
+  <joint name="right_wheel_joint" type="continuous">
+    <origin xyz="0.136 0.1 0.07" rpy="0 -1.5708 0" />
+    <parent link="base_link" />
+    <child link="right_wheel_1" />
+    <axis xyz="0.0 0.0 1.0" />
+  </joint>
+  <link name="right_wheel_1">
+    <inertial>
+      <origin xyz="0.138452 0.100000 0.070000" rpy="0 1.5708 0" />
+      <mass value="1.24" />
+      <inertia ixx="2.678055e-03" iyy="1.655421e-03" izz="1.655420e-03"
+        ixy="-1.010053e-12" iyz="5.132002e-11"
+        ixz="-4.656754e-13" />
+    </inertial>
+    <visual>
+      <origin xyz="-0.07 -0.1 0.136" rpy="0 1.5708 0" />
+      <geometry>
+        <mesh filename="package://megarover_description/meshes/mega3/right_wheel_1.stl" scale="0.001 0.001 0.001" />
+      </geometry>
+      <material name="dark_grey" />
+    </visual>
+    <collision>
+      <origin xyz="-0.07 -0.1 0.136" rpy="0 1.5708 0" />
+      <geometry>
+        <mesh filename="package://megarover_description/meshes/mega3/right_wheel_1.stl" scale="0.001 0.001 0.001" />
+      </geometry>
+    </collision>
+  </link>
 </robot>
