Commit message: xacro/urdfの修正

File: urdf/f120a.xacro (robot description, xacro)
@@ -3,18 +3,20 @@
   <xacro:include filename="$(find megarover_description)/urdf/materials.xacro" />
   <xacro:include filename="$(find megarover_description)/urdf/f120a.gazebo" />
-  <xacro:include filename="$(find megarover_description)/urdf/f120a_ros2_control.xacro" />
+  <xacro:arg name="use_ros2_control" default="true" />
+  <xacro:if value="$(arg use_ros2_control)">
+    <xacro:include filename="$(find megarover_description)/urdf/f120a_ros2_control.xacro" />
+  </xacro:if>
   <!-- OPTION  LRF TG30 -->
-  <!--<xacro:include filename="$(find vs_rover_options_description)/urdf/lrf/tg30_f120a.xacro" />-->
+  <!-- <xacro:include filename="$(find vs_rover_options_description)/urdf/lrf/tg30_f120a.xacro" />-->
   <!-- OPTION  bumper sensor -->
   <!-- <xacro:include filename="$(find vs_rover_options_description)/urdf/bumper/bumper_f120a.xacro" />
-  <xacro:bumperbaseboard prefix="front" parent="base_link" xyz="0 ${0.272 + bumper_alu_frame_y_offset} 0.0385" z_dir="180" />
-  <xacro:bumperbaseboard prefix="back" parent="base_link" xyz="0 ${-0.272 + bumper_alu_frame_y_offset} 0.0385" z_dir="0" /> -->
-  <!-- OPTION  camera stay -->
-  <!-- <xacro:include filename="$(find vs_rover_options_description)/urdf/cam_stay/cam_stay_f120a.xacro" /> -->
+  <xacro:bumperbaseboard prefix="front" parent="base_link" xyz="${0.272 + bumper_alu_frame_y_offset} 0 0.0385" z_dir="90" />
+  <xacro:bumperbaseboard prefix="back" parent="base_link" xyz="${-0.272 + bumper_alu_frame_y_offset} 0 0.0385" z_dir="-90" />-->
   <!-- OPTION  Intel Realsense depth camera D435i (camera stay is required)  -->
-  <!-- <xacro:include filename="$(find vs_rover_options_description)/urdf/depth_cam/_d435i.urdf.xacro" />
+  <!-- <xacro:include filename="$(find vs_rover_options_description)/urdf/cam_stay/cam_stay_f120a.xacro" />
+  <xacro:include filename="$(find vs_rover_options_description)/urdf/depth_cam/_d435i.urdf.xacro" />
   <xacro:sensor_d435i parent="cam_mount_link" use_nominal_extrinsics="true">
     <origin xyz="0.0295 0 0.0095" rpy="0 0 0" />
-  </xacro:sensor_d435i> -->
+  </xacro:sensor_d435i>-->
   <!-- OPTION  AMIR 740 (disabled by default because of interference with camera stay)-->
   <!-- <xacro:include filename="$(find amir_description)/urdf/amir_for_rover.xacro" />
@@ -28,16 +30,16 @@
     <parent link="base_footprint" />
     <child link="base_link" />
-    <origin xyz="-0.108 0 0" rpy="0 0 -1.5708" />
+    <origin xyz="-0.108 0 0" rpy="0 0 0" />
   </joint>
   <link name="base_link">
     <inertial>
-      <origin xyz="-0.000002 -0.012552 0.124849" rpy="0 0 0" />
+      <origin xyz="-0.012552 0.000002 0.124849" rpy="0 0 0" />
       <mass value="26.5" />
-      <inertia ixx="3.703059e-01" iyy="2.862913e-01" izz="5.773479e-01"
-        ixy="1.109256e-05" iyz="4.327049e-03"
-        ixz="-8.886529e-07" />
+      <inertia ixx="2.862913e-01" iyy="3.703059e-01" izz="5.773479e-01"
+        ixy="-1.109256e-05" iyz="8.886529e-07"
+        ixz="4.327049e-03" />
     </inertial>
     <visual>
-      <origin xyz="0 0 0" rpy="0 0 0" />
+      <origin xyz="0 0 0" rpy="0 0 -1.5708" />
       <geometry>
         <mesh filename="package://megarover_description/meshes/f120a/base_link.stl" scale="0.001 0.001 0.001" />
@@ -46,5 +48,5 @@
     </visual>
     <collision>
-      <origin xyz="0 0 0" rpy="0 0 0" />
+      <origin xyz="0 0 0" rpy="0 0 -1.5708" />
       <geometry>
         <mesh filename="package://megarover_description/meshes/f120a/base_link.stl" scale="0.001 0.001 0.001" />
@@ -53,19 +55,19 @@
   </link>
   <joint name="right_wheel_joint" type="continuous">
-    <origin xyz="0.202 0.108 0.085" rpy="0 -1.5708 0" />
+    <origin xyz="0.108 -0.202 0.085" rpy="0 0 0" />
     <parent link="base_link" />
     <child link="right_wheel_1" />
-    <axis xyz="0.0 0.0 1.0" />
+    <axis xyz="0.0 1.0 0.0" />
   </joint>
   <link name="right_wheel_1">
     <inertial>
-      <origin xyz="0.204466 0.108001 0.085004" rpy="0 0 0" />
+      <origin xyz="0 0 0" rpy="0 0 0" />
       <mass value="3.3" />
-      <inertia ixx="1.037325e-02" iyy="6.022157e-03" izz="6.021823e-03"
-        ixy="3.443741e-09" iyz="-1.410248e-07"
-        ixz="3.078066e-08" />
+      <inertia ixx="6.647813e-03" iyy="1.192125e-02" izz="6.647813e-03"
+        ixy="0.0" iyz="0.0"
+        ixz="0.0" />
     </inertial>
     <visual>
-      <origin xyz="-0.085 -0.108 0.202" rpy="0 1.5708 0" />
+      <origin xyz="-0.108 0.202 -0.085" rpy="0 0 -1.5708" />
       <geometry>
         <mesh filename="package://megarover_description/meshes/f120a/right_wheel_1.stl" scale="0.001 0.001 0.001" />
@@ -74,26 +76,26 @@
     </visual>
     <collision>
-      <origin xyz="-0.085 -0.108 0.202" rpy="0 1.5708 0" />
+      <origin xyz="0 0 0" rpy="1.5708 0 0" />
       <geometry>
-        <mesh filename="package://megarover_description/meshes/f120a/right_wheel_1.stl" scale="0.001 0.001 0.001" />
+        <cylinder radius="0.085" length="0.05" />
       </geometry>
     </collision>
   </link>
   <joint name="left_wheel_joint" type="continuous">
-    <origin xyz="-0.202 0.108 0.085" rpy="0 -1.5708 0" />
+    <origin xyz="0.108 0.202 0.085" rpy="0 0 0" />
     <parent link="base_link" />
     <child link="left_wheel_1" />
-    <axis xyz="0.0 0.0 1.0" />
+    <axis xyz="0.0 1.0 0.0" />
   </joint>
   <link name="left_wheel_1">
     <inertial>
-      <origin xyz="-0.204466 0.108004 0.085001" rpy="0 0 0" />
+      <origin xyz="0 0 0" rpy="0 0 0" />
       <mass value="3.3" />
-      <inertia ixx="1.037325e-02" iyy="6.021823e-03" izz="6.022157e-03"
-        ixy="-3.081416e-08" iyz="-1.410216e-07"
-        ixz="-3.441302e-09" />
+      <inertia ixx="6.647813e-03" iyy="1.192125e-02" izz="6.647813e-03"
+        ixy="0.0" iyz="0.0"
+        ixz="0.0" />
     </inertial>
     <visual>
-      <origin xyz="-0.085 -0.108 -0.202" rpy="0 1.5708 0" />
+      <origin xyz="-0.108 -0.202 -0.085" rpy="0 0 -1.5708" />
       <geometry>
         <mesh filename="package://megarover_description/meshes/f120a/left_wheel_1.stl" scale="0.001 0.001 0.001" />
@@ -102,7 +104,7 @@
     </visual>
     <collision>
-      <origin xyz="-0.085 -0.108 -0.202" rpy="0 1.5708 0" />
+      <origin xyz="0 0 0" rpy="1.5708 0 0" />
       <geometry>
-        <mesh filename="package://megarover_description/meshes/f120a/left_wheel_1.stl" scale="0.001 0.001 0.001" />
+        <cylinder radius="0.085" length="0.05" />
       </geometry>
     </collision>

File: urdf/mega3.xacro (robot description, xacro)
@@ -3,11 +3,14 @@
   <xacro:include filename="$(find megarover_description)/urdf/materials.xacro" />
   <xacro:include filename="$(find megarover_description)/urdf/mega3.gazebo" />
-  <xacro:include filename="$(find megarover_description)/urdf/mega3_ros2_control.xacro" />
+  <xacro:arg name="use_ros2_control" default="true" />
+  <xacro:if value="$(arg use_ros2_control)">
+    <xacro:include filename="$(find megarover_description)/urdf/mega3_ros2_control.xacro" />
+  </xacro:if>
   <!-- OPTION LRF TG30 -->
-  <xacro:include filename="$(find vs_rover_options_description)/urdf/lrf/tg30_mega3.xacro" />
+  <!-- <xacro:include filename="$(find vs_rover_options_description)/urdf/lrf/tg30_mega3.xacro" />-->
   <!-- OPTION  bumper sensor -->
   <!-- <xacro:include filename="$(find vs_rover_options_description)/urdf/bumper/bumper_mega3.xacro" />
-  <xacro:bumperbaseboard prefix="front" parent="base_link" xyz="0 0.19 0.02" z_dir="180" />
-  <xacro:bumperbaseboard prefix="back" parent="base_link" xyz="0 -0.19 0.02" z_dir="0" /> -->
+  <xacro:bumperbaseboard prefix="front" parent="base_link" xyz="0.19 0 0.02" z_dir="90" />
+  <xacro:bumperbaseboard prefix="back" parent="base_link" xyz="-0.19 0 0.02" z_dir="-90" />-->
   <!-- OPTION  camera stay -->
   <!-- <xacro:include filename="$(find vs_rover_options_description)/urdf/cam_stay/cam_stay_mega3.xacro" />
@@ -15,28 +18,28 @@
   <xacro:sensor_d435i parent="cam_mount_link" use_nominal_extrinsics="true">
     <origin xyz="0.0295 0 0.0095" rpy="0 0 0" />
-  </xacro:sensor_d435i> -->
+  </xacro:sensor_d435i>-->
   <!-- OPTION  AMIR 740 (disabled by default because of interference with camera stay)-->
   <!-- <xacro:include filename="$(find amir_description)/urdf/amir_for_rover.xacro" />
   <joint name="base_fixed" type="fixed">
-    <origin xyz="0.0 0.03 0.398" rpy="0 0 0" />
+    <origin xyz="0.03 0.0 0.398" rpy="0 0 -1.5708" />
     <parent link="base_link" />
     <child link="link0_1" />
-  </joint> -->
+  </joint>-->
   <link name="base_footprint" />
   <joint name="base_joint" type="fixed">
     <parent link="base_footprint" />
     <child link="base_link" />
-    <origin xyz="-0.1 0 0" rpy="0 0 -1.5708" />
+    <origin xyz="-0.1 0 0" rpy="0 0 0" />
   </joint>
   <link name="base_link">
     <inertial>
-      <origin xyz="0.000146 -0.000007 0.095171" rpy="0 0 0" />
+      <origin xyz="-0.000007 -0.000146 0.095171" rpy="0 0 0" />
       <mass value="12" />
-      <inertia ixx="9.308603e-02" iyy="5.644759e-02" izz="1.250700e-01"
-        ixy="3.125032e-04" iyz="-2.464583e-03"
-        ixz="2.117978e-05" />
+      <inertia ixx="5.644759e-02" iyy="9.308603e-02" izz="1.250700e-01"
+        ixy="-3.125032e-04" iyz="-2.117978e-05"
+        ixz="-2.464583e-03" />
     </inertial>
     <visual>
-      <origin xyz="0 0 0" rpy="0 0 0" />
+      <origin xyz="0 0 0" rpy="0 0 -1.5708" />
       <geometry>
         <mesh filename="package://megarover_description/meshes/mega3/base_link.stl" scale="0.001 0.001 0.001" />
@@ -45,5 +48,5 @@
     </visual>
     <collision>
-      <origin xyz="0 0 0" rpy="0 0 0" />
+      <origin xyz="0 0 0" rpy="0 0 -1.5708" />
       <geometry>
         <mesh filename="package://megarover_description/meshes/mega3/base_link.stl" scale="0.001 0.001 0.001" />
@@ -52,19 +55,19 @@
   </link>
   <joint name="left_wheel_joint" type="continuous">
-    <origin xyz="-0.136 0.1 0.07" rpy="0 -1.5708 0" />
+    <origin xyz="0.1 0.136 0.07" rpy="0 0 0" />
     <parent link="base_link" />
     <child link="left_wheel_1" />
-    <axis xyz="0.0 0.0 1.0" />
+    <axis xyz="0.0 1.0 0.0" />
   </joint>
   <link name="left_wheel_1">
     <inertial>
-      <origin xyz="-0.138454 0.100000 0.070000" rpy="0 0 0" />
+      <origin xyz="0 0 0" rpy="0 0 0" />
       <mass value="1.24" />
-      <inertia ixx="2.678186e-03" iyy="1.655435e-03" izz="1.655435e-03"
-        ixy="2.305704e-12" iyz="-5.140092e-11"
-        ixz="5.431314e-14" />
+      <inertia ixx="1.655435e-03" iyy="2.678186e-03" izz="1.655435e-03"
+        ixy="0.0" iyz="0.0"
+        ixz="0.0" />
     </inertial>
     <visual>
-      <origin xyz="-0.07 -0.1 -0.136" rpy="0 1.5708 0" />
+      <origin xyz="-0.1 -0.136 -0.07" rpy="0 0 -1.5708" />
       <geometry>
         <mesh filename="package://megarover_description/meshes/mega3/left_wheel_1.stl" scale="0.001 0.001 0.001" />
@@ -73,26 +76,26 @@
     </visual>
     <collision>
-      <origin xyz="-0.07 -0.1 -0.136" rpy="0 1.5708 0" />
+      <origin xyz="0 0 0" rpy="-1.5708 0 0" />
       <geometry>
-        <mesh filename="package://megarover_description/meshes/mega3/left_wheel_1.stl" scale="0.001 0.001 0.001" />
+        <cylinder radius="0.07" length="0.05" />
       </geometry>
     </collision>
   </link>
   <joint name="right_wheel_joint" type="continuous">
-    <origin xyz="0.136 0.1 0.07" rpy="0 -1.5708 0" />
+    <origin xyz="0.1 -0.136 0.07" rpy="0 0 0" />
     <parent link="base_link" />
     <child link="right_wheel_1" />
-    <axis xyz="0.0 0.0 1.0" />
+    <axis xyz="0.0 1.0 0.0" />
   </joint>
   <link name="right_wheel_1">
     <inertial>
-      <origin xyz="0.138452 0.100000 0.070000" rpy="0 1.5708 0" />
+      <origin xyz="0 0 0" rpy="0 0 0" />
       <mass value="1.24" />
-      <inertia ixx="2.678055e-03" iyy="1.655421e-03" izz="1.655420e-03"
-        ixy="-1.010053e-12" iyz="5.132002e-11"
-        ixz="-4.656754e-13" />
+      <inertia ixx="1.655421e-03" iyy="2.678055e-03" izz="1.655420e-03"
+        ixy="0.0" iyz="0.0"
+        ixz="0.0" />
     </inertial>
     <visual>
-      <origin xyz="-0.07 -0.1 0.136" rpy="0 1.5708 0" />
+      <origin xyz="-0.1 0.136 -0.07" rpy="0 0 -1.5708" />
       <geometry>
         <mesh filename="package://megarover_description/meshes/mega3/right_wheel_1.stl" scale="0.001 0.001 0.001" />
@@ -101,7 +104,7 @@
     </visual>
     <collision>
-      <origin xyz="-0.07 -0.1 0.136" rpy="0 1.5708 0" />
+      <origin xyz="0 0 0" rpy="-1.5708 0 0" />
       <geometry>
-        <mesh filename="package://megarover_description/meshes/mega3/right_wheel_1.stl" scale="0.001 0.001 0.001" />
+        <cylinder radius="0.07" length="0.05" />
       </geometry>
     </collision>

File: urdf/s40a_lb.xacro (robot description, xacro)
@@ -3,24 +3,10 @@
   <xacro:include filename="$(find megarover_description)/urdf/materials.xacro" />
   <xacro:include filename="$(find megarover_description)/urdf/s40a_lb.gazebo" />
-  <xacro:include filename="$(find megarover_description)/urdf/s40a_lb_ros2_control.xacro" />
+  <xacro:arg name="use_ros2_control" default="true" />
+  <xacro:if value="$(arg use_ros2_control)">
+    <xacro:include filename="$(find megarover_description)/urdf/s40a_lb_ros2_control.xacro" />
+  </xacro:if>
   <!-- OPTION LRF TG30 -->
-  <!--<xacro:include filename="$(find vs_rover_options_description)/urdf/lrf/tg30_s40a_lb.xacro" />-->
-  <!-- OPTION  bumper sensor -->
-  <!-- <xacro:include filename="$(find vs_rover_options_description)/urdf/bumper/bumper_s40a_lb.xacro" />
-  <xacro:bumperbaseboard prefix="front" parent="base_link" xyz="0 0.19 0.02" z_dir="180" />
-  <xacro:bumperbaseboard prefix="back" parent="base_link" xyz="0 -0.19 0.02" z_dir="0" /> -->
-  <!-- OPTION  camera stay -->
-  <!-- <xacro:include filename="$(find vs_rover_options_description)/urdf/cam_stay/cam_stay_s40a_lb.xacro" />
-  <xacro:include filename="$(find vs_rover_options_description)/urdf/depth_cam/_d435i.urdf.xacro" />
-  <xacro:sensor_d435i parent="cam_mount_link" use_nominal_extrinsics="true">
-    <origin xyz="0.0295 0 0.0095" rpy="0 0 0" />
-  </xacro:sensor_d435i> -->
-  <!-- OPTION  AMIR 740 (disabled by default because of interference with camera stay)-->
-  <!-- <xacro:include filename="$(find amir_description)/urdf/amir_for_rover.xacro" />
-  <joint name="base_fixed" type="fixed">
-    <origin xyz="0.0 0.03 0.398" rpy="0 0 0" />
-    <parent link="base_link" />
-    <child link="link0_1" />
-  </joint> -->
+  <xacro:include filename="$(find vs_rover_options_description)/urdf/lrf/tg30_s40a_lb.xacro" />
   <!-- sus.stl -->
   <xacro:macro name="sus_stl">
@@ -166,10 +152,12 @@
   <link name="base_link">
     <inertial>
-      <origin xyz="-0.000020 -0.001921 0.135459"/>
+      <origin xyz="-0.001921 0.000020 0.135459"/>
       <mass value="18.000000"/>
       <inertia
-        ixx="2.652700e-01" iyy="1.502132e-01" izz="2.510547e-01"
-        ixy="1.843531e-03" iyz="1.989196e-03" ixz="-4.115150e-04"/>
-    </inertial>
+        ixx="1.502132e-01" iyy="2.652700e-01" izz="2.510547e-01"
+        ixy="-1.843531e-03" iyz="4.115150e-04" ixz="1.989196e-03"/>
+    </inertial>
+  </link>
+  <link name="body_link">
     <visual>
       <geometry>
@@ -214,7 +202,14 @@
   <xacro:macro name="base_fixed_joint">
     <joint name="base_joint" type="fixed">
-      <origin xyz="0 0 0" rpy="0 0 -1.5708"/>
+      <origin xyz="0 0 0" rpy="0 0 0"/>
       <parent link="base_footprint"/>
       <child link="base_link"/>
+    </joint>
+  </xacro:macro>
+  <xacro:macro name="body_fixed_joint">
+    <joint name="body_joint" type="fixed">
+      <origin xyz="0 0 0" rpy="0 0 -1.5708"/>
+      <parent link="base_link"/>
+      <child link="body_link"/>
     </joint>
   </xacro:macro>
@@ -282,14 +277,15 @@
   <!-- ================================================== -->
   <xacro:base_fixed_joint/>
+  <xacro:body_fixed_joint/>
   <!-- drive -->
   <xacro:drive_sus_joint
     name="left_sus_joint"
     xyz="-0.119 0 0.051" rpy="0 0 ${radians(180)}"
-    parent="base_link"
+    parent="body_link"
     child="left_sus"/>
   <xacro:drive_sus_joint
     name="right_sus_joint"
     xyz="0.119 0 0.051" rpy="0 0 0"
-    parent="base_link"
+    parent="body_link"
     child="right_sus"/>
   <xacro:drive_wheel_joint
@@ -311,20 +307,20 @@
     name="front_left_caster_sus_joint"
     xyz="-0.165 0.13 0.082" rpy="0 0 0"
-    parent="base_link"
+    parent="body_link"
     child="front_left_caster_sus"/>
   <xacro:caster_sus_joint
     name="front_right_caster_sus_joint"
     xyz="0.165 0.13 0.082" rpy="0 0 0"
-    parent="base_link"
+    parent="body_link"
     child="front_right_caster_sus"/>
   <xacro:caster_sus_joint
     name="back_right_caster_sus_joint"
     xyz="0.165 -0.13 0.082" rpy="0 0 ${radians(180)}"
-    parent="base_link"
+    parent="body_link"
     child="back_right_caster_sus"/>
   <xacro:caster_sus_joint
     name="back_left_caster_sus_joint"
     xyz="-0.165 -0.13 0.082" rpy="0 0 ${radians(180)}"
-    parent="base_link"
+    parent="body_link"
     child="back_left_caster_sus"/>
   <!-- caster steering -->
@@ -369,10 +365,10 @@
     name="front_lrf_mount"
     xyz="0.0 0.0 0.0" rpy="0 0 ${radians(0)}"
-    parent="base_link"
+    parent="body_link"
     child="front_lrf_mount"/>
   <xacro:s40a_lb_lrf_mount_joint
     name="back_lrf_mount"
     xyz="0.0 0.0 0.0" rpy="0 0 ${radians(180)}"
-    parent="base_link"
+    parent="body_link"
     child="back_lrf_mount"/>
 </robot>
